File: drive4/_saved_drive4.sch (KiCad schematic (older format))
At the start: 7 parts, among them IC1 ATMEGA328-A

Commit message: a
Parts:
- removed C? (x2): C, symbol C
- removed IC1: ATMEGA328-A, TQFP32, symbol ATMEGA328-A
- removed Q? (x3): IRF7343PBF, SO-8, symbol IRF7343PBF
- removed Y?: Crystal_Small, symbol Crystal_Small
- added U?: ATMEGA328-AU, Housings_QFP:TQFP-32_7x7mm_Pitch0.8mm, symbol ATMEGA328-AU
Connections:
- net labels removed: GND
- wire segments 15 -> 0
Changed lines of the file:
@@
 encoding utf-8
 Sheet 1 1
-Title "Четырехканальный драйвер двигателей"
+Title ""
 Date ""
 Rev ""
@@
 $EndDescr
 $Comp
-L ATMEGA328-A IC1
-U 1 1 58A7ED6E
-P 3300 2650
-F 0 "IC1" H 2550 3900 50  0000 L BNN
-F 1 "ATMEGA328-A" H 3700 1250 50  0000 L BNN
-F 2 "TQFP32" H 3300 2650 50  0000 C CIN
-F 3 "" H 3300 2650 50  0000 C CNN
-	1    3300 2650
+L ATMEGA328-AU U?
+U 1 1 5A271A97
+P 3750 3500
+F 0 "U?" H 3000 4750 50  0000 L BNN
+F 1 "ATMEGA328-AU" H 4150 2100 50  0000 L BNN
+F 2 "Housings_QFP:TQFP-32_7x7mm_Pitch0.8mm" H 3750 3500 50  0001 C CIN
+F 3 "" H 3750 3500 50  0001 C CNN
+	1    3750 3500
 	1    0    0    -1
 $EndComp
-Wire Wire Line
-	2300 3950 2300 3650
-Wire Wire Line
-	2300 3650 2400 3650
-Wire Wire Line
-	2300 3750 2400 3750
-Connection ~ 2300 3750
-Wire Wire Line
-	2400 3850 2300 3850
-Connection ~ 2300 3850
-$Comp
-L IRF7343PBF Q?
-U 1 1 58A7F1F8
-P 7150 3750
-F 0 "Q?" H 7400 3825 50  0000 L CNN
-F 1 "IRF7343PBF" H 7400 3750 50  0000 L CNN
-F 2 "SO-8" H 7400 3675 50  0000 L CNN
-F 3 "" H 7150 3750 50  0000 L CNN
-	1    7150 3750
-	1    0    0    -1
-$EndComp
-$Comp
-L IRF7343PBF Q?
-U 2 1 58A7F23F
-P 5550 3500
-F 0 "Q?" H 5800 3575 50  0000 L CNN
-F 1 "IRF7343PBF" H 5800 3500 50  0000 L CNN
-F 2 "SO-8" H 5800 3425 50  0000 L CNN
-F 3 "" H 5550 3500 50  0000 L CNN
-	2    5550 3500
-	1    0    0    -1
-$EndComp
-$Comp
-L GND #PWR?
-U 1 1 58A7F53F
-P 2300 3950
-F 0 "#PWR?" H 2300 3700 50  0001 C CNN
-F 1 "GND" H 2300 3800 50  0000 C CNN
-F 2 "" H 2300 3950 50  0000 C CNN
-F 3 "" H 2300 3950 50  0000 C CNN
-	1    2300 3950
-	1    0    0    -1
-$EndComp
-$Comp
-L IRF7343PBF Q?
-U 1 1 58A7F7DA
-P 6350 2150
-F 0 "Q?" H 6600 2225 50  0000 L CNN
-F 1 "IRF7343PBF" H 6600 2150 50  0000 L CNN
-F 2 "SO-8" H 6600 2075 50  0000 L CNN
-F 3 "" H 6350 2150 50  0000 L CNN
-	1    6350 2150
-	1    0    0    -1
-$EndComp
-Wire Wire Line
-	4300 2250 4450 2250
-Wire Wire Line
-	4450 2250 4450 2400
-Wire Wire Line
-	4450 2400 4800 2400
-Wire Wire Line
-	4300 2150 4450 2150
-Wire Wire Line
-	4450 2150 4450 2000
-Wire Wire Line
-	4450 2000 4800 2000
-$Comp
-L C C?
-U 1 1 58A7F960
-P 4950 2000
-F 0 "C?" H 4975 2100 50  0000 L CNN
-F 1 "C" H 4975 1900 50  0000 L CNN
-F 2 "" H 4988 1850 50  0000 C CNN
-F 3 "" H 4950 2000 50  0000 C CNN
-	1    4950 2000
-	0    1    1    0
-$EndComp
-$Comp
-L C C?
-U 1 1 58A7F9FF
-P 4950 2400
-F 0 "C?" H 4975 2500 50  0000 L CNN
-F 1 "C" H 4975 2300 50  0000 L CNN
-F 2 "" H 4988 2250 50  0000 C CNN
-F 3 "" H 4950 2400 50  0000 C CNN
-	1    4950 2400
-	0    1    1    0
-$EndComp
-Connection ~ 4700 2400
-Connection ~ 4700 2000
-Wire Wire Line
-	5100 2400 5200 2400
-Wire Wire Line
-	5200 2400 5200 2000
-Wire Wire Line
-	5200 2000 5100 2000
-$Comp
-L GND #PWR?
-U 1 1 58A7FA5B
-P 5200 2200
-F 0 "#PWR?" H 5200 1950 50  0001 C CNN
-F 1 "GND" H 5200 2050 50  0000 C CNN
-F 2 "" H 5200 2200 50  0000 C CNN
-F 3 "" H 5200 2200 50  0000 C CNN
-	1    5200 2200
-	0    -1   -1   0
-$EndComp
-$Comp
-L Crystal_Small Y?
-U 1 1 58A7FB29
-P 4700 2200
-F 0 "Y?" H 4700 2300 50  0000 C CNN
-F 1 "Crystal_Small" H 4700 2100 50  0000 C CNN
-F 2 "" H 4700 2200 50  0000 C CNN
-F 3 "" H 4700 2200 50  0000 C CNN
-	1    4700 2200
-	0    1    1    0
-$EndComp
-Wire Wire Line
-	4700 2100 4700 2000
-Wire Wire Line
-	4700 2300 4700 2400
 $EndSCHEMATC
