File: drive4/drive4.kicad_pcb (KiCad board)
At the start: 2 copper layers, 1 part, among them Q0 IRF7343PBF

Commit message: a
Parts:
- removed Q0: IRF7343PBF, SO-8
- added C1: C, Capacitors_SMD:C_0402, F.Cu at (141.0, 82.5)
- added C2: C, Capacitors_SMD:C_0402, F.Cu at (163.8, 81.3)
- added C3: C, Capacitors_SMD:C_0402, F.Cu at (139.7, 91.4)
- added J1: FTDI Port, Pin_Headers:Pin_Header_Angled_1x06_Pitch1.00mm, F.Cu at (133.3, 86.4)
- added R1: R, Resistors_SMD:R_0402, F.Cu at (137.2, 77.5)
- added U1: ATMEGA328-AU, Housings_QFP:TQFP-32_7x7mm_Pitch0.8mm, F.Cu at (147.3, 86.4)
- added Y1: Crystal_GND2, Crystals:Crystal_SMD_FOX_FQ7050-4pin_7.0x5.0mm, F.Cu at (160.0, 92.7)
Routing:
- net GND: track 0.00 -> 12.1 mm
- net VCC: track 0.00 -> 4.23 mm
