File: drive4/drive4.sch (KiCad schematic (older format))
At the start: 2 parts, among them IC1 ATMEGA328-A, Q0 IRF7343PBF

Commit message: a
Parts:
- removed IC1: ATMEGA328-A, TQFP32, symbol ATMEGA328-A
- removed Q0: IRF7343PBF, SO-8, symbol IRF7343PBF
- added C1, C2, C3: C, Capacitors_SMD:C_0402, symbol C
- added J1: FTDI Port, Pin_Headers:Pin_Header_Angled_1x06_Pitch1.00mm, symbol Conn_01x06
- added R1: R, Resistors_SMD:R_0402, symbol R
- added U1: ATMEGA328-AU, Housings_QFP:TQFP-32_7x7mm_Pitch0.8mm, symbol ATMEGA328-AU
- added Y1: Crystal_GND2, Crystals:Crystal_SMD_FOX_FQ7050-4pin_7.0x5.0mm, symbol Crystal_GND2
Connections:
- net labels added: A0, A1, A2, A3, A6, A7, D10, D2, D3, D4, D5, D6, D7, D8, D9, DTR, GND, MISO, MOSI, RESET, RX, SCK, SCL, SDA, TX, VCC
- net labels removed: Earth
- wire segments 4 -> 19
- no-connect marks 0 -> 20
